Commit message: Broadcasting de tf setpoint au lieu d'envoyer des commandes de vitesse. Renaming des nom de tf::frames.

File: elikos_navigation_stack/elikos_nav/cfg/flying_box.urdf.xacro (robot description, xacro)
@@ -1,4 +1,4 @@
 <robot name="flying_box">
-  <link name="base_link">
+  <link name="elikos_base_link">
     <visual>
       <origin xyz="0 0 0" rpy="0 0 0" />

Commit message: Le modèle du drone est maintenant un cylindre. Vérification que le point envoyé est plus loin qu'une certaine distance de tolérance.

File: elikos_navigation_stack/elikos_nav/cfg/flying_box.urdf.xacro (robot description, xacro)
@@ -4,5 +4,5 @@
       <origin xyz="0 0 0" rpy="0 0 0" />
       <geometry>
-          <box size="0.25 0.25 0.25"/>
+          <cylinder length="0.3" radius="0.3"/>
       </geometry>
     </visual>

Commit message: L execution de la trajectoire et l evitement d obstacle semblent fonctionnnels. Il reste a decider quand faire un clear_octomap.

File: elikos_navigation_stack/elikos_nav/cfg/flying_box.urdf.xacro (robot description, xacro)
@@ -4,5 +4,5 @@
       <origin xyz="0 0 0" rpy="0 0 0" />
       <geometry>
-          <cylinder length="0.3" radius="0.3"/>
+          <sphere radius="0.3"/>
       </geometry>
     </visual>

Commit message: Taille du modele spherique, ajout de launch files globaux et integration du AI.

File: elikos_navigation_stack/elikos_nav/cfg/flying_box.urdf.xacro (robot description, xacro)
@@ -4,5 +4,5 @@
       <origin xyz="0 0 0" rpy="0 0 0" />
       <geometry>
-          <sphere radius="0.3"/>
+          <sphere radius="0.44"/>
       </geometry>
     </visual>
